File: ep2c35_trial/ep2c35_trial.kicad_sch (KiCad schematic)
At the start: 5 parts, among them U1 EP2C5F484

Commit message: EP2C35 trial. WIP.
Parts:
- added J1, J2: Conn_02x21_Odd_Even, Connector_PinHeader_1.27mm:PinHeader_2x21_P1.27mm_Horizontal, symbol Connector_Generic:Conn_02x21_Odd_Even
- added J3: 3M_8540-4500PL, logic_analyzer:3M_8540-4500PL, symbol logic_analyzer:3M_8540-4500PL
- added R11, R12, R13, R14, R15, R16, R17, R18, R19, R20, R21, R22, R23, R24, R25, R26, R27, R28, R29, R30: 100, Resistor_SMD:R_0402_1005Metric, symbol Device:R
- added U2: XC6SLX16-FTG256, Package_BGA:Xilinx_FTG256, symbol FPGA_Xilinx_Spartan6:XC6SLX16-FTG256
- added U3: FT600Q-B-T, logic_analyzer:QFN-56-1EP_7x7mm_P0.4mm_FT600Q, symbol logic_analyzer:FT600Q-B-T
Connections:
- net +2V5: no longer U1.A2 (VCCIO3), U1.A21 (VCCIO4), U1.B1 (VCCIO2), U1.B22 (VCCIO5), U1.C11 (VCCIO3), U1.C12 (VCCIO4), U1.C6 (VCCIO3), U1.D17 (VCCIO4), U1.E10 (VCCIO3), U1.E13 (VCCIO4), U1.G14 (VCCIO4), U1.G19 (VCCIO5), U1.G9 (VCCIO3), U1.J16 (VCCIO5), U1.J7 (VCCIO2), U1.L20 (VCCIO5), U1.L3 (VCCIO2)
- net GNDD: now also U1.M22 (CLK6/LVDSCLK3p/input), J1.1 (Pin_1), J1.10 (Pin_10), J1.12 (Pin_12), J1.14 (Pin_14), J1.16 (Pin_16), J1.18 (Pin_18), J1.2 (Pin_2), J1.20 (Pin_20), J1.22 (Pin_22), J1.24 (Pin_24), J1.26 (Pin_26), J1.28 (Pin_28), J1.30 (Pin_30), J1.32 (Pin_32), J1.34 (Pin_34), J1.36 (Pin_36), J1.38 (Pin_38), J1.4 (Pin_4), J1.40 (Pin_40), J1.42 (Pin_42), J1.6 (Pin_6), J1.8 (Pin_8), J2.1 (Pin_1), J2.10 (Pin_10), J2.12 (Pin_12), J2.14 (Pin_14), J2.16 (Pin_16), J2.18 (Pin_18), J2.2 (Pin_2), J2.20 (Pin_20), J2.22 (Pin_22), J2.24 (Pin_24), J2.26 (Pin_26), J2.28 (Pin_28), J2.30 (Pin_30), J2.32 (Pin_32), J2.34 (Pin_34), J2.36 (Pin_36), J2.38 (Pin_38), J2.4 (Pin_4), J2.40 (Pin_40), J2.41 (Pin_41), J2.42 (Pin_42), J2.6 (Pin_6), J2.8 (Pin_8), R20.2
- net FT_WR_N: now reaches U1.A10 (IO/LVDS70p)
- net FT_WR_N: now also U3.7 (WR_N)
- net FT_OE_N: now reaches U1.A11 (IO/LVDS73p)
- net FT_OE_N: now also U3.9 (OE_N)
- net FT_DATA7: now reaches U1.A3 (IO/LVDS50p)
- net FT_DATA7: now also U3.42 (DATA_7)
- net FT_DATA8: now reaches U1.A4 (IO/LVDS51p)
- net FT_DATA8: now also U3.45 (DATA_8)
- net FT_DATA10: now reaches U1.A5 (IO/LVDS52p)
- net FT_DATA10: now also U3.47 (DATA_10)
- net FT_DATA12: now reaches U1.A6 (IO/LVDS53p)
- net FT_DATA12: now also U3.53 (DATA_12)
- net FT_DATA14: now reaches U1.A7 (IO/LVDS61p)
- net FT_DATA14: now also U3.55 (DATA_14)
- net FT_BE0: now reaches U1.A8 (IO/LVDS62p)
- net FT_BE0: now also U3.2 (BE_0)
- net FT_TXE_N: now reaches U1.A9 (IO/LVDS67p)
- net FT_TXE_N: now also U3.4 (TXE_N)
- net FT_RD_N: now reaches U1.B10 (IO/LVDS70n)
- net FT_RD_N: now also U3.8 (RD_N)
- net FT_RESET_N: now reaches U1.B11 (IO/LVDS73n)
- net FT_RESET_N: now also U3.10 (RESET_N)
- net FT_CLK: now reaches U1.B3 (IO/DEV_CLRn/LVDS50n)
- net FT_CLK: now also U3.43 (CLK)
- net FT_DATA9: now reaches U1.B4 (IO/LVDS51n)
- net FT_DATA9: now also U3.46 (DATA_9)
- net FT_DATA11: now reaches U1.B5 (IO/LVDS52n)
- net FT_DATA11: now also U3.48 (DATA_11)
- net FT_DATA13: now reaches U1.B6 (IO/LVDS53n)
- net FT_DATA13: now also U3.54 (DATA_13)
- net FT_DATA15: now reaches U1.B7 (IO/LVDS61n)
- net FT_DATA15: now also U3.56 (DATA_15)
- net FT_BE1: now reaches U1.B8 (IO/LVDS62n)
- net FT_BE1: now also U3.3 (BE_1)
- net FT_RXF_N: now reaches U1.B9 (IO/LVDS67n)
- net FT_RXF_N: now also U3.5 (RXF_N)
- net FT_GPIO1: now reaches U1.C10 (IO/VREFB3N0)
- net FT_GPIO1: now also U3.13 (GPIO1)
- net FT_WAKEUP_N: now reaches U1.C9 (IO/LVDS59p)
- net FT_WAKEUP_N: now also U3.11 (WAKEUP_N)
- net FT_GPIO0: now reaches U1.D9 (IO/LVDS64p)
- net FT_GPIO0: now also U3.12 (GPIO0)
- net FT_DATA5: now reaches U1.C1 (IO/LVDS47p)
- net FT_DATA5: now also U3.40 (DATA_5)
- net FT_DATA6: now reaches U1.C2 (IO/LVDS47n)
- net FT_DATA6: now also U3.41 (DATA_6)
- net FT_DATA3: now reaches U1.D1 (IO/LVDS40p)
- net FT_DATA3: now also U3.36 (DATA_3)
- net FT_DATA4: now reaches U1.D2 (IO/LVDS40n)
- net FT_DATA4: now also U3.39 (DATA_4)
- net FT_DATA1: now reaches U1.E1 (IO/LVDS37p)
- net FT_DATA1: now also U3.34 (DATA_1)
- net FT_DATA2: now reaches U1.E2 (IO/LVDS37n)
- net FT_DATA2: now also U3.35 (DATA_2)
- net FT_DATA0: now reaches U1.F2 (IO/LVDS36n)
- net FT_DATA0: now also U3.33 (DATA_0)
- net LVDS_RX_CLK0_P: now reaches U1.M1 (CLK2/LVDSCLK1p/input)
- net LVDS_RX_CLK0_P: now also J1.41 (Pin_41), R30.2
- net LVDS_RX_CLK0_N: now reaches U1.M2 (CLK3/LVDSCLK1n/input)
- net LVDS_RX_CLK0_N: now also J1.39 (Pin_39), R30.1
- net at U1.M5 (IO/LVDS26p): now also U1.M6 (IO/LVDS26n)
- net at U1.M7 (IO/LVDS23n): now also U1.M8 (IO/LVDS23p)
- net LVDS_RX_DATA0_0_P: now reaches U1.N1 (IO/LVDS25p)
- net LVDS_RX_DATA0_0_P: now also J1.37 (Pin_37), R28.2
- net LVDS_RX_DATA0_0_N: now reaches U1.N2 (IO/LVDS25n)
- net LVDS_RX_DATA0_0_N: now also J1.35 (Pin_35), R28.1
- net at U1.N3 (IO/LVDS20p): now also U1.N4 (IO/LVDS20n)
- net at U1.N5 (IO/LVDS22n): now also U1.N6 (IO/LVDS22p)
- net LVDS_RX_DATA0_1_P: now reaches U1.P1 (IO/LVDS24p)
- net LVDS_RX_DATA0_1_P: now also J1.33 (Pin_33), R27.2
- net LVDS_RX_DATA0_1_N: now reaches U1.P2 (IO/LVDS24n)
- net LVDS_RX_DATA0_1_N: now also J1.31 (Pin_31), R27.1
- net at U1.P4 (IO/LVDS12p): now also U1.R4 (IO/LVDS12n)
- net at U1.P5 (IO/LVDS17p): now also U1.P6 (IO/LVDS17n)
- net LVDS_RX_DATA0_2_P: now reaches U1.R1 (IO/LVDS16p)
- net LVDS_RX_DATA0_2_P: now also J1.29 (Pin_29), R26.2
- net LVDS_RX_DATA0_2_N: now reaches U1.R2 (IO/LVDS16n)
- net LVDS_RX_DATA0_2_N: now also J1.27 (Pin_27), R26.1
- net at U1.R5 (IO/LVDS10p): now also U1.R6 (IO/LVDS10n)
- net at U1.R7 (IO/LVDS18n): now also U1.R8 (IO/LVDS18p)
- net LVDS_RX_DATA0_3_P: now reaches U1.T1 (IO/LVDS13p)
- net LVDS_RX_DATA0_3_P: now also J1.25 (Pin_25), R25.2
- net LVDS_RX_DATA0_3_N: now reaches U1.T2 (IO/LVDS13n)
- net LVDS_RX_DATA0_3_N: now also J1.23 (Pin_23), R25.1
- net at U1.T5 (IO/LVDS7p): now also U1.T6 (IO/LVDS7n)
- net LVDS_RX_DATA0_4_P: now reaches U1.U1 (IO/LVDS11p)
- net LVDS_RX_DATA0_4_P: now also J1.21 (Pin_21), R24.2
- net LVDS_RX_DATA0_4_N: now reaches U1.U2 (IO/LVDS11n)
- net LVDS_RX_DATA0_4_N: now also J1.19 (Pin_19), R24.1
- net LVDS_RX_DATA0_5_P: now reaches U1.V1 (IO/LVDS8p)
- net LVDS_RX_DATA0_5_P: now also J1.17 (Pin_17), R23.2
- net LVDS_RX_DATA0_5_N: now reaches U1.V2 (IO/LVDS8n)
- net LVDS_RX_DATA0_5_N: now also J1.15 (Pin_15), R23.1
- net LVDS_RX_DATA0_6_P: now reaches U1.W1 (IO/LVDS6p)
- net LVDS_RX_DATA0_6_P: now also J1.13 (Pin_13), R22.2
- net LVDS_RX_DATA0_6_N: now reaches U1.W2 (IO/LVDS6n)
- net LVDS_RX_DATA0_6_N: now also J1.11 (Pin_11), R22.1
- net at U1.W3 (IO/LVDS2p): now also U1.W4 (IO/LVDS2n)
- net LVDS_RX_DATA0_7_P: now reaches U1.Y1 (IO/LVDS5p)
- net LVDS_RX_DATA0_7_P: now also J1.9 (Pin_9), R21.2
- net LVDS_RX_DATA0_7_N: now reaches U1.Y2 (IO/LVDS5n)
- net LVDS_RX_DATA0_7_N: now also J1.7 (Pin_7), R21.1
- net LVDS_RX_FCLK0_P: now reaches U1.Y3 (IO/LVDS0p)
- net LVDS_RX_FCLK0_P: now also J1.5 (Pin_5), R29.2
- net LVDS_RX_FCLK0_N: now reaches U1.Y4 (IO/LVDS0n)
- net LVDS_RX_FCLK0_N: now also J1.3 (Pin_3), R29.1
- net LVDS_RX_CLK1_N: now reaches U1.M21 (CLK7/LVDSCLK3n/input)
- net LVDS_RX_CLK1_N: now also J2.39 (Pin_39), R20.1
- net LVDS_RX_DATA1_7_N: now reaches U1.N21 (IO/LVDS128n)
- net LVDS_RX_DATA1_7_N: now also J2.3 (Pin_3), R11.1
- net LVDS_RX_DATA1_7_P: now reaches U1.N22 (IO/LVDS128p)
- net LVDS_RX_DATA1_7_P: now also J2.5 (Pin_5), R11.2
- net LVDS_RX_DATA1_6_N: now reaches U1.P21 (IO/LVDS129n)
- net LVDS_RX_DATA1_6_N: now also J2.7 (Pin_7), R12.1
- net LVDS_RX_DATA1_6_P: now reaches U1.P22 (IO/LVDS129p)
- net LVDS_RX_DATA1_6_P: now also J2.9 (Pin_9), R12.2
- net LVDS_RX_DATA1_5_N: now reaches U1.R21 (IO/LVDS134n)
- net LVDS_RX_DATA1_5_N: now also J2.11 (Pin_11), R13.1
- net LVDS_RX_DATA1_5_P: now reaches U1.R22 (IO/LVDS134p)
- net LVDS_RX_DATA1_5_P: now also J2.13 (Pin_13), R13.2
- net LVDS_RX_DATA1_4_N: now reaches U1.T21 (IO/LVDS135n)
- net LVDS_RX_DATA1_4_N: now also J2.15 (Pin_15), R14.1
- net LVDS_RX_DATA1_4_P: now reaches U1.T22 (IO/LVDS135p)
- net LVDS_RX_DATA1_4_P: now also J2.17 (Pin_17), R14.2
- net LVDS_RX_DATA1_3_N: now reaches U1.U21 (IO/LVDS139n)
- net LVDS_RX_DATA1_3_N: now also J2.19 (Pin_19), R15.1
- net LVDS_RX_DATA1_3_P: now reaches U1.U22 (IO/LVDS139p)
- net LVDS_RX_DATA1_3_P: now also J2.21 (Pin_21), R15.2
- net LVDS_RX_DATA1_2_N: now reaches U1.V21 (IO/LVDS140n)
- net LVDS_RX_DATA1_2_N: now also J2.23 (Pin_23), R16.1
- net LVDS_RX_DATA1_2_P: now reaches U1.V22 (IO/LVDS140p)
- net LVDS_RX_DATA1_2_P: now also J2.25 (Pin_25), R16.2
- net LVDS_RX_DATA1_1_N: now reaches U1.W21 (IO/LVDS145n)
- net LVDS_RX_DATA1_1_N: now also J2.27 (Pin_27), R17.1
- net LVDS_RX_DATA1_1_P: now reaches U1.W22 (IO/LVDS145p)
- net LVDS_RX_DATA1_1_P: now also J2.29 (Pin_29), R17.2
- net LVDS_RX_FCLK1_N: now reaches U1.Y19 (IO/LVDS149n)
- net LVDS_RX_FCLK1_N: now also J2.35 (Pin_35), R19.1
- net LVDS_RX_FCLK1_P: now reaches U1.Y20 (IO/LVDS149p)
- net LVDS_RX_FCLK1_P: now also J2.37 (Pin_37), R19.2
- net LVDS_RX_DATA1_0_N: now reaches U1.Y21 (IO/LVDS141n)
- net LVDS_RX_DATA1_0_N: now also J2.31 (Pin_31), R18.1
- net LVDS_RX_DATA1_0_P: now reaches U1.Y22 (IO/LVDS141p)
- net LVDS_RX_DATA1_0_P: now also J2.33 (Pin_33), R18.2
- new net +3.3V: U1.A2 (VCCIO3), U1.A21 (VCCIO4), U1.B1 (VCCIO2), U1.B22 (VCCIO5), U1.C11 (VCCIO3), U1.C12 (VCCIO4), U1.C6 (VCCIO3), U1.D17 (VCCIO4), U1.E10 (VCCIO3), U1.E13 (VCCIO4), U1.G14 (VCCIO4), U1.G19 (VCCIO5), U1.G9 (VCCIO3), U1.J16 (VCCIO5), U1.J7 (VCCIO2), U1.L20 (VCCIO5), U1.L3 (VCCIO2)
- new net FT_SIWU_N: U3.6 (SIWU_N)
Other:
- moved on the sheet: C3, C4, U1F, U1G, U1H, U1I

Commit message: Wire up FTDI FT600Q.
Parts:
- added C10, C11, C12, C13, C14, C16, C17, C18, C9: 100n, Capacitor_SMD:C_0402_1005Metric, symbol Device:C
- added C5, C6, C7: 0.1u, Capacitor_SMD:C_0402_1005Metric, symbol Device:C
- added C8: 4.7u, Capacitor_SMD:C_0402_1005Metric, symbol Device:C
- added FB1, FB2: BLM18PG221SN1D, Resistor_SMD:R_0603_1608Metric, symbol Device:FerriteBead
- added J4: USB3_B_Micro_Amphenol_GSB343K331HR, Amphenol_GSB343K331HR:AMPHENOL_GSB343K331HR, symbol logic_analyzer:USB3_B_Micro_Amphenol_GSB343K331HR
- added R1: 1.6k/1%, Resistor_SMD:R_0402_1005Metric, symbol Device:R
Connections:
- net GNDA is gone; now on net GNDD: U1.V7 (GNDA_PLL1)
- net +3.3V: now also U3.15 (VCC33), U3.19 (VCC33), U3.22 (VDDA), U3.30 (VCC33), U3.38 (VCCIO), U3.44 (VCCIO), U3.52 (VCCIO), C10.2, C11.2, C12.2, C13.2, C14.2, C9.2
- net GNDD: now also U3.32 (GND), U3.49 (GND), U3.51 (GND), U3.57 (GND), C10.1, C11.1, C12.1, C13.1, C14.1, C16.1, C17.1, C18.1, C5.2, C8.1, C9.1, FB2.2, J4.5 (GND), J4.8 (DRAIN), R1.2; no longer J2.41 (Pin_41), R20.2, U1.M22 (CLK6/LVDSCLK3p/input)
- net +1V0: now reaches U3.1 (AVDD)
- net +1V0: now also U3.23 (VD10), U3.26 (VD10), U3.31 (DV10), U3.37 (VD10), U3.50 (VD10), C16.2, C17.2, C18.2, C8.2
- net USB_D_N: now reaches U3.18 (DP)
- net USB_D_N: now also J4.2 (D-)
- net USB_D_P: now reaches U3.20 (DM)
- net USB_D_P: now also J4.3 (D+)
- net USB_RREF: now reaches U3.21 (RREF)
- net USB_RREF: now also R1.1
- net USB_SSTX_N: now reaches U3.24 (TODN)
- net USB_SSTX_N: now also C6.2
- net USB_SSTX_P: now reaches U3.25 (TODP)
- net USB_SSTX_P: now also C7.2
- net USB_SSRX_N: now reaches U3.27 (RIDN)
- net USB_SSRX_N: now also J4.9 (SSRX-)
- net USB_SSRX_P: now reaches U3.28 (RIDP)
- net USB_SSRX_P: now also J4.10 (SSRX+)
- net VBUS: now reaches U3.29 (VBUS)
- net VBUS: now also FB1.1
- net at U1.P3 (IO/VREFB1N0): now also U1.T3 (IO)
- net at U1.U3 (IO/VREFB1N1): now also U1.U4 (IO/PLL1_OUTp)
- net at U1.V4 (IO/PLL1_OUTn): now also U1.W5 (IO)
- new net LVDS_RX_CLK1_P: J2.41 (Pin_41), R20.2, U1.M22 (CLK6/LVDSCLK3p/input)
- new net USB_SHIELD: FB2.1, J4.S1 (SHIELD), J4.S2 (SHIELD)
- new net USB_SSTX_RAW_N: C6.1, J4.6 (SSTX-)
- new net USB_SSTX_RAW_P: C7.1, J4.7 (SSTX+)
- new net VBUS_RAW: C5.1, FB1.2, J4.1 (VBUS)
- no-connect marks 0 -> 1
Other:
- moved on the sheet: U3

Commit message: Before switching to hierarchical sheets.
Parts:
- added C15: 100n, Capacitor_SMD:C_0402_1005Metric, symbol Device:C
- added J5: Conn_02x05_Odd_Even, Connector_PinHeader_2.54mm:PinHeader_2x05_P2.54mm_Vertical, symbol Connector_Generic:Conn_02x05_Odd_Even
- added R2, R3, R4, R5, R6: 10K, Resistor_SMD:R_0402_1005Metric, symbol Device:R
- added TP1: TestPoint, TestPoint:TestPoint_Pad_D1.0mm, symbol Connector:TestPoint
- added U4: W25Q16JVSNIQ, Package_SO:SOIC-8_5.23x5.23mm_P1.27mm, symbol logic_analyzer:W25Q16JVSNIQ
Connections:
- net +2V5: now also R5.1, R6.1
- net +3.3V: now also C15.2, J5.4 (Pin_4), R2.1, R3.2, R4.2, U4.8 (VCC)
- net GNDD: now also J3.10 (GND), J3.12 (GND), J3.14 (GND), J3.16 (GND), J3.18 (GND), J3.2 (PGND), J3.20 (GND), J3.22 (GND), J3.24 (GND), J3.26 (GND), J3.28 (GND), J3.30 (GND), J3.32 (GND), J3.34 (GND), J3.36 (GND), J3.38 (GND), J3.4 (GND), J3.40 (PGND), J3.6 (GND), J3.8 (GND), U1.K1 (nCE), U1.M17 (MSEL0), U1.N17 (MSEL1), C15.1, J5.10 (Pin_10), J5.2 (Pin_2), U4.4 (GND)
- net +5V: now reaches J3.1 (+5V)
- net +5V: now also J3.39 (+5V)
- net POD_D13: now reaches J3.11 (D13)
- net POD_D12: now reaches J3.13 (D12)
- net POD_D11: now reaches J3.15 (D11)
- net POD_D10: now reaches J3.17 (D10)
- net POD_D9: now reaches J3.19 (D9)
- net POD_D8: now reaches J3.21 (D8)
- net POD_D7: now reaches J3.23 (D7)
- net POD_D6: now reaches J3.25 (D6)
- net POD_D5: now reaches J3.27 (D5)
- net POD_D4: now reaches J3.29 (D4)
- net POD_CLK: now reaches J3.3 (CLOCK)
- net POD_D3: now reaches J3.31 (D3)
- net POD_D2: now reaches J3.33 (D2)
- net POD_D1: now reaches J3.35 (D1)
- net POD_D0: now reaches J3.37 (D0)
- net POD_D15: now reaches J3.7 (D15)
- net POD_D14: now reaches J3.9 (D14)
- net SPI_nCS: now reaches U1.C3 (IO/nCSO)
- net SPI_nCS: now also U4.1 (~{CS})
- net SPI_ADS: now reaches U1.C4 (IO/ASDO)
- net SPI_ADS: now also U4.5 (DI(IO0))
- net CRC_ERROR: now reaches U1.D3 (IO/CRC_ERROR/LVDS49p)
- net CRC_ERROR: now also TP1.1
- net TCK: now reaches U1.K2 (TCK)
- net TCK: now also J5.1 (Pin_1)
- net SPI_DATA0: now reaches U1.K4 (DATA0)
- net SPI_DATA0: now also U4.2 (DO(IO1))
- net TDI: now reaches U1.K5 (TDI)
- net TDI: now also J5.9 (Pin_9)
- net TMS: now reaches U1.K6 (TMS)
- net TMS: now also J5.5 (Pin_5)
- net at U1.L4 (nCONFIG): now also R2.2
- net TDO: now reaches U1.L5 (TDO)
- net TDO: now also J5.3 (Pin_3)
- net SPI_DCLK: now reaches U1.L6 (DCLK)
- net SPI_DCLK: now also U4.6 (CLK)
- net LVDS26: now reaches U1.M5 (IO/LVDS26p), U1.M6 (IO/LVDS26n)
- net LVDS23: now reaches U1.M7 (IO/LVDS23n), U1.M8 (IO/LVDS23p)
- net LVDS20: now reaches U1.N3 (IO/LVDS20p), U1.N4 (IO/LVDS20n)
- net LVDS22: now reaches U1.N5 (IO/LVDS22n), U1.N6 (IO/LVDS22p)
- net LVDS12: now reaches U1.P4 (IO/LVDS12p), U1.R4 (IO/LVDS12n)
- net LVDS17: now reaches U1.P5 (IO/LVDS17p), U1.P6 (IO/LVDS17n)
- net LVDS10: now reaches U1.R5 (IO/LVDS10p), U1.R6 (IO/LVDS10n)
- net LVDS18: now reaches U1.R7 (IO/LVDS18n), U1.R8 (IO/LVDS18p)
- net LVDS7: now reaches U1.T5 (IO/LVDS7p), U1.T6 (IO/LVDS7n)
- net LVDS2: now reaches U1.W3 (IO/LVDS2p), U1.W4 (IO/LVDS2n)
- net CONF_DONE: now reaches U1.N18 (CONF_DONE)
- net CONF_DONE: now also R6.2
- net nSTATUS: now reaches U1.N20 (nSTATUS)
- net nSTATUS: now also R5.2
- new net SPI_nRESET: R4.1, U4.7 (IO3)
- new net SPI_nWP: R3.1, U4.3 (IO2)
- no-connect marks 1 -> 5
Other:
- added sheet EP2C35 (ep2c35.kicad_sch)
- moved on the sheet: J3, U2A, U2B, U2C, U2D

Commit message: Fix tons of ERC violations.
Parts:
- removed U2: XC6SLX16-FTG256, Package_BGA:Xilinx_FTG256, symbol FPGA_Xilinx_Spartan6:XC6SLX16-FTG256
- added C19, C20: 18p, Capacitor_SMD:C_0402_1005Metric, symbol Device:C
- added C21: 4.7u, Capacitor_SMD:C_0402_1005Metric, symbol Device:C
- added R7: 10k, Resistor_SMD:R_0402_1005Metric, symbol Device:R
- added Y1: ABM7-30.000MHZ-D2Y-T, Crystal:Crystal_SMD_0603-2Pin_6.0x3.5mm_HandSoldering, symbol Device:Crystal
Connections:
- net +5V is gone; now on net VBUS: J3.1 (+5V), J3.39 (+5V)
- net +3.3V: now also C21.2, R7.2
- net FT_SIWU_N: now also R7.1
- net GNDD: now also C19.1, C20.1, C21.1
- net at U3.16 (XI): now also C20.2, Y1.2
- net at U3.17 (XO): now also C19.2, Y1.1
- no-connect marks 5 -> 230
Other:
- moved on the sheet: C13, C14, R1

Commit message: Power supplies.
Parts:
- added C22: 100n, Capacitor_SMD:C_0402_1005Metric, symbol Device:C
- added C23, C25: 2u, Capacitor_SMD:C_0805_2012Metric, symbol Device:C
- added C24, C26: 47u, Capacitor_SMD:C_1206_3216Metric, symbol Device:C
- added C27, C28, C29: 1u, Capacitor_SMD:C_0805_2012Metric, symbol Device:C
- added J6, J7, J8: Conn_01x02_Male, Connector_PinHeader_2.54mm:PinHeader_1x02_P2.54mm_Vertical, symbol Connector:Conn_01x02_Male
- added R10, R31, R8, R9: 10k, Resistor_SMD:R_0402_1005Metric, symbol Device:R
- added U2: MIC37302, logic_analyzer:S-PAK-5, symbol logic_analyzer:MIC37302
- added U5: MIC39102, logic_analyzer:SOICN-8LD-PL-1, symbol logic_analyzer:MIC39102
- added U6: MIC49150-1.2, logic_analyzer:SOICN-8LD-PL-1, symbol logic_analyzer:MIC49150-1.2
- added X1: FNETHE025, Oscillator:Oscillator_SMD_IQD_IQXO70-4Pin_7.5x5.0mm, symbol logic_analyzer:FNETHE025
Connections:
- net +1V2: now also J8.2 (Pin_2)
- net +2V5: now also C28.2, J7.2 (Pin_2), U6.3 (VIN)
- net +3.3V: now also C22.2, C25.2, C27.2, J6.2 (Pin_2), U5.1 (EN), U5.2 (IN), U6.1 (EN), U6.2 (VBIAS), X1.4 (Vdd)
- net VBUS: now also C23.2, U2.1 (EN), U2.2 (VIN)
- net CLK25: now reaches U1.A12 (CLK9/LVDSCLK4p/input)
- net CLK25: now also X1.3 (OUT)
- net LVDS48: now reaches U1.E3 (IO/LVDS48p)
- net LVDS48: now also U1.E4 (IO/LVDS48n)
- net GNDD renamed GND
- net GND: now also C22.1, C23.1, C24.1, C25.1, C26.1, C27.1, C28.1, C29.1, R31.1, R9.1, U2.3 (GND), U5.5 (GND), U5.6 (GND), U5.7 (GND), U5.8 (GND), U6.5 (GND), U6.6 (GND), U6.7 (GND), U6.8 (GND), X1.2 (GND)
- new net 1V2_LDO: C29.2, J8.1 (Pin_1), U6.4 (VOUT)
- new net 2V5_ADJ: R10.1, R31.2, U5.4 (ADJ)
- new net 2V5_LDO: C26.2, J7.1 (Pin_1), R10.2, U5.3 (OUT)
- new net 3V3_ADJ: R8.1, R9.2, U2.5 (ADJ)
- new net 3V3_LDO: C24.2, J6.1 (Pin_1), R8.2, U2.4 (VOUT)
- no-connect marks 230 -> 229
Other:
- moved on the sheet: C1, C2

Commit message: Add digital interface. Power islands.
Parts:
- added C30: 10u, Capacitor_SMD:C_0805_2012Metric, symbol Device:C
- added C31, C33, C35: 1n, Capacitor_SMD:C_0402_1005Metric, symbol Device:C
- added C32, C34, C36, C37, C38, C39, C40, C41, C42, C43, C44, C45, C46, C47, C48, C49, C50, C51, C52, C53, C54, C55, C56, C57, C58, C59, C60, C61, C62, C63, C64, C65, C66, C67, C68, C69, C70: 100n, Capacitor_SMD:C_0402_1005Metric, symbol Device:C
- added FB3: BLM18PG221SN1D, Resistor_SMD:R_0603_1608Metric, symbol Device:FerriteBead
- added J9: Conn_01x02_Male, Connector_PinHeader_2.54mm:PinHeader_1x02_P2.54mm_Vertical, symbol Connector:Conn_01x02_Male
- added R32, R33, R34, R35, R36, R37, R38, R39, R40, R41, R42, R43, R44, R45, R46, R47, R48: 10k, Resistor_SMD:R_0402_1005Metric, symbol Device:R
Connections:
- net +1V2: now also C37.1, C38.1, C39.1, C40.1, C41.1, C42.1, C43.1, C44.1, C45.1, C46.1, C47.1, C48.1, C49.1, J9.1 (Pin_1)
- net +1V2A: now also C30.2, C31.1, C32.1, C33.1, C34.1, C35.1, C36.1, FB3.2
- net +2V5: now also C50.1, C51.1, C52.1, C53.1, C54.1, C55.1, C56.1, C57.1, C58.1, C59.1, C69.1
- net +3.3V: now also C60.1, C61.1, C62.1, C63.1, C64.1, C65.1, C66.1, C67.1, C68.1, C70.1
- net GND: now also C30.1, C31.2, C32.2, C33.2, C34.2, C35.2, C36.2, C37.2, C38.2, C39.2, C40.2, C41.2, C42.2, C43.2, C44.2, C45.2, C46.2, C47.2, C48.2, C49.2, C50.2, C51.2, C52.2, C53.2, C54.2, C55.2, C56.2, C57.2, C58.2, C59.2, C60.2, C61.2, C62.2, C63.2, C64.2, C65.2, C66.2, C67.2, C68.2, C69.2, C70.2
- net POD_CLK: now also R32.2
- net POD_D0: now also R48.2
- net POD_D1: now also R47.2
- net POD_D10: now also R38.2
- net POD_D11: now also R37.2
- net POD_D12: now also R36.2
- net POD_D13: now also R35.2
- net POD_D14: now also R34.2
- net POD_D15: now also R33.2
- net POD_D2: now also R46.2
- net POD_D3: now also R45.2
- net POD_D4: now also R44.2
- net POD_D5: now also R43.2
- net POD_D6: now also R42.2
- net POD_D7: now also R41.2
- net POD_D8: now also R40.2
- net POD_D9: now also R39.2
- net DIG_D0: now reaches U1.C21 (IO/LVDS104n)
- net DIG_D0: now also R48.1
- net DIG_D1: now reaches U1.C22 (IO/LVDS104p)
- net DIG_D1: now also R47.1
- net DIG_D2: now reaches U1.D21 (IO/LVDS108n)
- net DIG_D2: now also R46.1
- net DIG_D3: now reaches U1.D22 (IO/LVDS108p)
- net DIG_D3: now also R45.1
- net DIG_D4: now reaches U1.E21 (IO/LVDS109n)
- net DIG_D4: now also R44.1
- net DIG_D5: now reaches U1.E22 (IO/LVDS109p)
- net DIG_D5: now also R43.1
- net DIG_D6: now reaches U1.F21 (IO/LVDS112n)
- net DIG_D6: now also R42.1
- net DIG_D7: now reaches U1.F22 (IO/LVDS112p)
- net DIG_D7: now also R41.1
- net DIG_D8: now reaches U1.G21 (IO/LVDS114n)
- net DIG_D8: now also R40.1
- net DIG_D9: now reaches U1.G22 (IO/LVDS114p)
- net DIG_D9: now also R39.1
- net DIG_D10: now reaches U1.H21 (IO/LVDS122n)
- net DIG_D10: now also R38.1
- net DIG_D11: now reaches U1.H22 (IO/LVDS122p)
- net DIG_D11: now also R37.1
- net DIG_D12: now reaches U1.J21 (IO/LVDS124n)
- net DIG_D12: now also R36.1
- net DIG_D13: now reaches U1.J22 (IO/LVDS124p)
- net DIG_D13: now also R35.1
- net DIG_D14: now reaches U1.K21 (IO/LVDS125n)
- net DIG_D14: now also R34.1
- net DIG_D15: now reaches U1.K22 (IO/LVDS125p)
- net DIG_D15: now also R33.1
- net DIG_CLK: now reaches U1.L22 (CLK4/LVDSCLK2p/input)
- net DIG_CLK: now also R32.1
- new net 1V2_OPT: FB3.1, J9.2 (Pin_2)
- no-connect marks 229 -> 212
Other:
- moved on the sheet: J3, J8
