File: ep2c35_trial/ep2c35_trial.kicad_pcb (KiCad board)
At the start: 4 copper layers, 84.4 x 57.6 mm, 181 parts, among them J1 Conn_02x21_Odd_Even, J10 Conn_02x10_Odd_Even, J11 Conn_01x03_Pin, J2 Conn_02x21_Odd_Even, J3 3M_8540-4500PL, J4 USB3_B_Micro_Amphenol_GSB343K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, J5 Conn_02x05_Odd_Even, J7 Conn_01x03_Pin, J8 Conn_01x02_Male, J9 Conn_01x02_Male, U1 EP2C5F484, U10 SRV05-4, U11 SRV05-4, U12 LM317_TO-252, U13 LM317_TO-252, U17 SRV05-4, U2 MIC37302, U3 FT600Q-B-T, U4 W25Q16JVSNIQ, U5 MIC39102, U6 MIC49150-1.2, U7 SP3003-02UTG, U8 SRV05-4, U9 SRV05-4, X1 FNETHE025, Y1 ABM7-30.000MHZ-D2Y-T

Commit message: Rename EP2C5 to EP2C35.
Parts:
- U1: value EP2C5F484 -> EP2C35F484
