File: logic_analyzer/logic_analyzer.kicad_pcb (KiCad board)
At the start: 2 copper layers, 183 parts, among them J1 3M_8540-4500PL, U1 TLV3601, U10 TLV3601, U11 TLV3601, U12 ADA4891-4, U13 TLV3601, U14 TLV3601, U2 TLV3601, U3 ADA4891-4, U4 ADA4891-4, U5 ADA4891-4, U6 TLV3601, U7 TLV3601, U8 ADA4891-4, U9 ADA4891-4

Commit message: Unknown logic_analyzer changes.
Parts:
- C1, C10, C11, C12, C13, C14, C15, C16, C17, C18, C19, C2, C20, C21, C22, C23, C24, C25, C26, C27, C28, C29, C3, C30, C31, C32, C33, C34, C35, C36, C37, C38, C39, C4, C40, C41, C42, C43, C44, C45, C46, C47, C48, C49, C5, C50, C51, C52, C53, C54, C55, C56, C57, C58, C59, C6, C60, C61, C62, C63, C64, C65, C66, C67, C68, C69, C7, C70, C71, C72, C8, C9: footprint Capacitor_SMD:C_0603_1608Metric_Pad1.08x0.95mm_HandSolder -> Capacitor_SMD:C_0402_1005Metric
- R1, R10, R11, R12, R13, R14, R15, R16, R17, R18, R19, R2, R20, R21, R22, R23, R24, R25, R26, R27, R28, R29, R3, R30, R31, R32, R33, R34, R35, R36, R37, R38, R39, R4, R40, R41, R42, R43, R44, R45, R46, R47, R48, R49, R5, R50, R51, R52, R53, R54, R55, R56, R57, R58, R59, R6, R60, R61, R62, R63, R64, R65, R66, R67, R68, R69, R7, R70, R71, R72, R73, R74, R75, R76, R77, R78, R79, R8, R80, R81, R82, R83, R84, R85, R86, R87, R88, R9: footprint Resistor_SMD:R_0603_1608Metric_Pad0.98x0.95mm_HandSolder -> Resistor_SMD:R_0402_1005Metric
- moved C29 134.1 mm to (212.9, 101.6)
- moved C30 134.1 mm to (214.4, 101.6)
- moved C31 134.1 mm to (215.9, 101.6)
- moved U5 134.1 mm to (213.8, 78.5)
- moved R37 89.4 mm to (210.0, 90.0)
- moved U6 89.4 mm to (214.5, 87.8)
- moved R6 60.3 mm to (71.5, 98.7), turned to 180 degrees
- moved R10 57.4 mm to (71.5, 101.7), turned to 180 degrees
- moved C26 50.4 mm to (229.8, 95.6)
- moved C28 50.4 mm to (234.2, 90.5)
- moved C32 50.4 mm to (249.1, 74.5)
- moved C33 50.4 mm to (229.8, 98.1)
- moved C35 50.4 mm to (238.6, 77.9)
- moved R31 50.4 mm to (236.8, 82.9)
- moved R35 50.4 mm to (229.8, 90.5)
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Connections:
- net Net-(R10-Pad2) renamed /Input Section/OA4_out
- net Net-(R11-Pad1) renamed /Input Section/OA1_out
- net Net-(R12-Pad1) renamed /Input Section/OA2_out
- net Net-(R13-Pad1) renamed /Input Section/OA3_out
- net Net-(R31-Pad1) renamed /Input Section1/OA1_out
- net Net-(R33-Pad2) renamed /Input Section1/OA2_out
- net Net-(R38-Pad1) renamed /Input Section1/OA3_out
- net Net-(R40-Pad2) renamed /Input Section1/OA4_out
- net Net-(R61-Pad1) renamed /Input Section2/OA1_out
- net Net-(R63-Pad2) renamed /Input Section2/OA2_out
- net Net-(R68-Pad1) renamed /Input Section2/OA3_out
- net Net-(R70-Pad2) renamed /Input Section2/OA4_out
- net Net-(R75-Pad1) renamed /Input Section3/OA1_out
- net Net-(R77-Pad2) renamed /Input Section3/OA2_out
- net Net-(R82-Pad1) renamed /Input Section3/OA3_out
- net Net-(R84-Pad2) renamed /Input Section3/OA4_out
- R18 pad 1: /POD_CLK -> /Voff_buf
- R22 pad 1: /POD_CLK -> /Voff_buf
- R26 pad 1: /POD_CLK -> /Voff_buf
- R30 pad 1: /POD_CLK -> /Voff_buf
- R48 pad 1: /POD_CLK -> /Voff_buf
- R52 pad 1: /POD_CLK -> /Voff_buf
- R56 pad 1: /POD_CLK -> /Voff_buf
- R60 pad 1: /POD_CLK -> /Voff_buf
Routing:
- net /BUF_OUT0: track 0.00 -> 13.6 mm
- net /Input Section/OA1_out: track 0.00 -> 12.5 mm
- net GNDA: track 0.00 -> 12.3 mm
- net /BUF_OUT3: track 0.00 -> 11.6 mm
- net /Input Section/OA2_out: track 0.00 -> 7.91 mm
- net /Input Section/OA4_out: track 0.00 -> 7.85 mm
- net Net-(U3B--): track 0.00 -> 7.80 mm
- net /pod_buf4/BUF_IN2: track 0.00 -> 6.90 mm
- net /pod_buf4/BUF_IN1: track 0.00 -> 6.87 mm
- net /pod_buf4/BUF_IN3: track 0.00 -> 5.72 mm
- net +5VA: track 0.00 -> 4.76 mm, vias 0 -> 1
- net /BUF_OUT2: track 0.00 -> 3.93 mm
- net /BUF_OUT1: track 0.00 -> 3.92 mm
- net Net-(U3A--): track 0.00 -> 3.89 mm
- net -5VA: track 0.00 -> 3.61 mm
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Other:
- copper layers 2 -> 4
