File: logic_analyzer/logic_analyzer.kicad_sch (KiCad schematic)
At the start: 10 parts, among them U2 ADA4891-4, U3 ADA4891-4

Commit message: Front-end placement exercise.
Parts:
- removed C10, C5, C6, C9: 100n, symbol Device:C
- removed C11, C12, C7, C8: 10u, symbol Device:C
- removed U2, U3: ADA4891-4, symbol logic_analyzer:ADA4891-4
- added J1: 3M_8540-4500PL, logic_analyzer:3M_8540-4500PL, symbol logic_analyzer:3M_8540-4500PL
Connections:
- net GNDA: now also J1.10 (GND), J1.12 (GND), J1.14 (GND), J1.16 (GND), J1.18 (GND), J1.20 (GND), J1.22 (GND), J1.24 (GND), J1.26 (GND), J1.28 (GND), J1.30 (GND), J1.32 (GND), J1.34 (GND), J1.36 (GND), J1.38 (GND), J1.4 (GND), J1.6 (GND), J1.8 (GND)
- new net +5V: J1.1 (+5V), J1.39 (+5V)
- new net GNDD: J1.2 (PGND), J1.40 (PGND)
- new net POD_CLK: J1.3 (CLOCK)
- new net POD_D0: J1.37 (D0)
- new net POD_D1: J1.35 (D1)
- new net POD_D10: J1.17 (D10)
- new net POD_D11: J1.15 (D11)
- new net POD_D12: J1.13 (D12)
- new net POD_D13: J1.11 (D13)
- new net POD_D14: J1.9 (D14)
- new net POD_D15: J1.7 (D15)
- new net POD_D2: J1.33 (D2)
- new net POD_D3: J1.31 (D3)
- new net POD_D4: J1.29 (D4)
- new net POD_D5: J1.27 (D5)
- new net POD_D6: J1.25 (D6)
- new net POD_D7: J1.23 (D7)
- new net POD_D8: J1.21 (D8)
- new net POD_D9: J1.19 (D9)
- no-connect marks 0 -> 1
Other:
- added sheet pod_buf4 (pod_buf4.kicad_sch)
- added sheet pod_buf5 (pod_buf4.kicad_sch)
- sheet Input Section ports: added ADC_IN0+, ADC_IN0-, ADC_IN1+, ADC_IN1-, BUF_OUT0, BUF_OUT1, DIG_OUT0, DIG_OUT1, Voffset2; removed ADC_IN+, ADC_IN-, D_IN, IN, Voffset
- sheet Input Section1 ports: added ADC_IN0+, ADC_IN0-, ADC_IN1+, ADC_IN1-, BUF_OUT0, BUF_OUT1, DIG_OUT0, DIG_OUT1, Voffset2; removed ADC_IN+, ADC_IN-, D_IN, IN, Voffset
- sheet Input Section2 ports: added ADC_IN0+, ADC_IN0-, ADC_IN1+, ADC_IN1-, BUF_OUT0, BUF_OUT1, DIG_OUT0, DIG_OUT1, Voffset2; removed ADC_IN+, ADC_IN-, D_IN, IN, Voffset
- sheet Input Section3 ports: added ADC_IN0+, ADC_IN0-, ADC_IN1+, ADC_IN1-, BUF_OUT0, BUF_OUT1, DIG_OUT0, DIG_OUT1, Voffset2; removed ADC_IN+, ADC_IN-, D_IN, IN, Voffset

Commit message: Before switching to hierarchical sheets.
Changed lines of the file:
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@@
     (stroke (width 0) (type default) (color 0 0 0 0))
   )
-  (wire (pts (xy 57.15 120.65) (xy 72.39 120.65))
+  (wire (pts (xy 59.69 120.65) (xy 72.39 120.65))
     (stroke (width 0) (type default) (color 0 0 0 0))
   )
@@
     (stroke (width 0) (type default) (color 0 0 0 0))
   )
-  (wire (pts (xy 57.15 146.05) (xy 72.39 146.05))
+  (wire (pts (xy 59.69 146.05) (xy 72.39 146.05))
     (stroke (width 0) (type default) (color 0 0 0 0))
   )
@@
     (effects (font (size 1.27 1.27)) (justify left bottom))
   )
-  (label "POD_CLK" (at 60.96 146.05 0)
-    (effects (font (size 1.27 1.27)) (justify left bottom))
-  )
   (label "POD_D1" (at 60.96 139.7 0)
     (effects (font (size 1.27 1.27)) (justify left bottom))
@@
     (effects (font (size 1.27 1.27)) (justify left bottom))
   )
-  (label "POD_CLK" (at 60.96 120.65 0)
-    (effects (font (size 1.27 1.27)) (justify left bottom))
-  )
   (label "POD_D3" (at 40.64 113.03 0)
     (effects (font (size 1.27 1.27)) (justify left bottom))
   )
+  (label "Voff_buf" (at 60.96 120.65 0)
+    (effects (font (size 1.27 1.27)) (justify left bottom))
+  )
   (label "POD_D14" (at 40.64 85.09 0)
     (effects (font (size 1.27 1.27)) (justify left bottom))
@@
   )
   (label "POD_D0" (at 60.96 142.24 0)
+    (effects (font (size 1.27 1.27)) (justify left bottom))
+  )
+  (label "Voff_buf" (at 60.96 146.05 0)
     (effects (font (size 1.27 1.27)) (justify left bottom))
   )
@@
       (reference "#PWR059") (unit 1) (value "GNDD") (footprint "")
     )
+    (path "/7ddedb78-112d-4441-8e1b-67fe311493d9/1be7da6b-fbf6-47e4-8e75-b0a9902ab227"
+      (reference "#PWR?") (unit 1) (value "-5VA") (footprint "")
+    )
+    (path "/2e028959-4a26-46e7-9f55-db9d44f14998/1be7da6b-fbf6-47e4-8e75-b0a9902ab227"
+      (reference "#PWR?") (unit 1) (value "-5VA") (footprint "")
+    )
     (path "/26454115-225f-4e87-8a6c-cb4f8b4d98fa/1be7da6b-fbf6-47e4-8e75-b0a9902ab227"
       (reference "#PWR?") (unit 1) (value "-5VA") (footprint "")
     )
-    (path "/2e028959-4a26-46e7-9f55-db9d44f14998/1be7da6b-fbf6-47e4-8e75-b0a9902ab227"
-      (reference "#PWR?") (unit 1) (value "-5VA") (footprint "")
-    )
     (path "/1f432fef-ef5d-4967-b3ea-d12b8a8ee2d0/1be7da6b-fbf6-47e4-8e75-b0a9902ab227"
       (reference "#PWR?") (unit 1) (value "-5VA") (footprint "")
     )
-    (path "/7ddedb78-112d-4441-8e1b-67fe311493d9/1be7da6b-fbf6-47e4-8e75-b0a9902ab227"
-      (reference "#PWR?") (unit 1) (value "-5VA") (footprint "")
+    (path "/7ddedb78-112d-4441-8e1b-67fe311493d9/7a2ea4ea-d61b-43f7-a9da-f8e5dab3abe4"
+      (reference "#PWR?") (unit 1) (value "+5VA") (footprint "")
     )
     (path "/26454115-225f-4e87-8a6c-cb4f8b4d98fa/7a2ea4ea-d61b-43f7-a9da-f8e5dab3abe4"
@@
       (reference "#PWR?") (unit 1) (value "+5VA") (footprint "")
     )
-    (path "/7ddedb78-112d-4441-8e1b-67fe311493d9/7a2ea4ea-d61b-43f7-a9da-f8e5dab3abe4"
-      (reference "#PWR?") (unit 1) (value "+5VA") (footprint "")
-    )
