File: logic_analyzer/pod_buf4.kicad_sch (KiCad schematic)
At the start: 25 parts, among them U4 ADA4891-4

Commit message: Before switching to hierarchical sheets.
Parts:
- renumbered C15 to C37, C16 to C38, C17 to C39, C18 to C40, C19 to C41, C20 to C42, C21 to C43, C22 to C44, R15 to R45, R16 to R46, R17 to R47, R18 to R48, R19 to R49, R20 to R50, R21 to R51, R22 to R52, R23 to R53, R24 to R54, R25 to R55, R26 to R56, R27 to R57, R28 to R58, R29 to R59, R30 to R60, U4 to U8

Commit message: Unknown logic_analyzer changes.
Parts:
- C37, C38, C39, C40, C41, C42, C43, C44: footprint Capacitor_SMD:C_0603_1608Metric_Pad1.08x0.95mm_HandSolder -> Capacitor_SMD:C_0402_1005Metric
- R45, R46, R47, R48, R49, R50, R51, R52, R53, R54, R55, R56, R57, R58, R59, R60: footprint Resistor_SMD:R_0603_1608Metric_Pad0.98x0.95mm_HandSolder -> Resistor_SMD:R_0402_1005Metric
